File: electronics/neg5supply/max636/max636.brd (EAGLE design)
At the start: 28.2 x 21.6 mm, 14 parts, among them J1 +V, J2 -V, J3 GND, J4 GND, U1 MAX636

Commit message: layout tweaks
Parts:
- removed VR1: (no value), bt_electromech:PV36W
- added ADJ: 10K, bt_electromech:35WR
- U1: device bt_regulator:PDIP8 -> bt_regulator:SO08
- moved C3 6.97 mm to (15.0, 11.7), turned to 90 degrees
- moved R4 4.99 mm to (17.0, 11.7), turned to 90 degrees
- moved C2 4.75 mm to (13.0, 11.7), turned to 90 degrees
- moved L1 3.57 mm to (15.0, 17.3)
- moved D1 3.57 mm to (10.2, 17.3)
- moved J2 3.30 mm to (22.9, 12.7)
- moved J3 3.30 mm to (22.9, 10.2)
- moved R3 1.98 mm to (19.1, 11.7), turned to 270 degrees
- moved C1 1.66 mm to (7.24, 17.1), turned to 90 degrees
- moved U1 1.37 mm to (8.38, 9.14), turned to 0 degrees
- moved U$1 0.25 mm to (6.60, 0.76)
Connections:
- net N$2: now also ADJ.1; no longer VR1.1
- net N$5: now also ADJ.2; no longer VR1.2
Routing:
- net N$2: track 7.73 -> 23.6 mm
- net N$1: track 18.7 -> 10.2 mm, vias 2 -> 0
- net VCC: track 17.3 -> 14.7 mm, vias 1 -> 0
- net N$6: track 11.7 -> 13.6 mm
- net N$3: track 20.2 -> 18.7 mm, vias 1 -> 2
- net N$5: track 3.35 -> 4.70 mm
Other:
- board size 28.2 x 21.6 mm -> 24.9 x 21.6 mm
- board text added: "R0.2"
